File: pcb/Miriball36.kicad_sch (KiCad schematic)
At the start: 45 parts, among them J2 MJ-4PP-9, SW1 SW_PUSH, SW10 SW_PUSH, SW11 SW_PUSH, SW12 SW_PUSH, SW13 SW_PUSH, SW14 SW_PUSH, SW15 SW_PUSH, SW16 SW_PUSH, SW17 SW_PUSH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

Commit message: add logo & pin for trackball
Parts:
- added OL1: OLED, yuuichi_kbd:OLED_4Pin, symbol kbd:OLED
Connections:
- net GND: now also OL1.4 (GND)
- net VCC: now also OL1.3 (VCC)
- net sda: now reaches U1.5 (2/D1/SDA)
- net sda: now also OL1.1 (SDA)
- net scl: now reaches U1.6 (3/D0/SCL)
- net scl: now also OL1.2 (SCL)
- no-connect marks 10 -> 8
